File: PCB/BlankingRelay_Base/BlankingRelay_Base.kicad_pcb (KiCad board)
At the start: 2 copper layers, 40 parts, among them J1 Barrel_Jack, J2 Blanking In, J3 JST 7, J4 JST 7, J5 JST 7, J6 JST 7, J7 JST 7, J8 JST 7, J9 JST 7, SW1 SW_Push_DPDT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

Commit message: update base board to include outline and some keepout areas
Routing:
- net 5V: track 497.4 -> 498.4 mm
Other:
- board outline added: 120.2 x 75.2 mm
