File: PCB/BlankingRelay_modular/BlankingRelay_Base.kicad_pcb (KiCad board)
At the start: 2 copper layers, 97.2 x 75.2 mm, 27 parts, among them J1 Barrel_Jack, J2 Blanking In, J3 Conn_01x02_Socket, J4 Conn_01x02_Socket, J5 Conn_01x02_Socket, J6 Conn_01x02_Socket, J7 5 Vin (optional), SW1 SW_Push_DPDT, SW2 SW_Push_DPDT, SW3 SW_Push_DPDT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

Commit message: minor bug correction
Parts:
- removed R98: 1k, Resistor_THT:R_Axial_DIN0309_L9.0mm_D3.2mm_P15.24mm_Horizontal
- removed R99: 330, Resistor_THT:R_Axial_DIN0309_L9.0mm_D3.2mm_P15.24mm_Horizontal
- added R5: 1k, Resistor_THT:R_Axial_DIN0309_L9.0mm_D3.2mm_P15.24mm_Horizontal, F.Cu at (54.8, 93.8)
- added R6: 330, Resistor_THT:R_Axial_DIN0309_L9.0mm_D3.2mm_P15.24mm_Horizontal, F.Cu at (54.8, 98.5)
- moved J1 2.59 mm to (48.0, 84.9)
Routing:
- net +9V: track 9.06 -> 6.78 mm
